File: Malenia.sch (KiCad schematic (older format))
At the start: 151 parts, among them SW2 Rotary_Encoder_Switch

Commit message: Fix duplex overlap matrix
Connections:
- net R6: now also D55.1 (K)
- net R7: no longer D55.1 (K)
Other:
- moved on the sheet: D55
Changed lines of the file:
@@
 L Device:D_Small D55
 U 1 1 62C3E803
-P 6250 4500
-F 0 "D55" V 6296 4430 50  0000 R CNN
-F 1 "SOD123" V 6205 4430 50  0000 R CNN
-F 2 "sanproject-keyboard-part:DIODE_1206_SawnsProjects" V 6250 4500 50  0001 C CNN
-F 3 "~" V 6250 4500 50  0001 C CNN
-	1    6250 4500
+P 6250 4450
+F 0 "D55" V 6296 4380 50  0000 R CNN
+F 1 "SOD123" V 6205 4380 50  0000 R CNN
+F 2 "sanproject-keyboard-part:DIODE_1206_SawnsProjects" V 6250 4450 50  0001 C CNN
+F 3 "~" V 6250 4450 50  0001 C CNN
+	1    6250 4450
 	0    -1   -1   0
 $EndComp
@@
 Wire Wire Line
 	5050 4300 5050 4400
-Wire Wire Line
-	6250 4300 6250 4400
 Wire Wire Line
 	1250 3300 1250 4100
@@
 Wire Wire Line
 	6250 2700 6250 2750
-Connection ~ 5850 2200
 Wire Wire Line
 	5850 1900 5850 2000
@@
 	5450 2150 6250 2150
 Connection ~ 6250 2150
-Wire Wire Line
-	5850 2200 6650 2200
 Wire Wire Line
 	6250 1900 6250 1950
@@
 Connection ~ 7250 3300
 Connection ~ 7250 4100
-Connection ~ 5850 4600
-Wire Wire Line
-	5850 4600 6250 4600
-Wire Wire Line
-	5450 4550 7050 4550
+Wire Wire Line
+	5450 4550 6250 4550
 Wire Wire Line
 	5850 4300 5850 4400
@@
 Text GLabel 7050 1900 0    50   Input ~ 0
 MX15
+Connection ~ 6250 4550
+Wire Wire Line
+	6250 4550 7050 4550
+Wire Wire Line
+	6250 4300 6250 4350
 $EndSCHEMATC
